File: Kicad_Project/CLK/CLK.sch (KiCad schematic (older format))
At the start: 7 parts

Commit message: CLK done
Parts:
- removed R?: 1k, symbol Device:R
- added C? (x2): 0.1 uF, symbol Device:C
- added C? (x3): 0.01 uF, symbol Device:C
- added R?: 1M, symbol Device:R
- added R? (x2): 1k, symbol Device:R
- added SW?: SW_Push, symbol Switch:SW_Push
- added SW?: SW_DPDT_x2, symbol Switch:SW_DPDT_x2
- added U? (x2): X, symbol newlib:X
- added U?: 74AHC1G32, symbol 74xGxx:74AHC1G32
- added U?: 74AHCT1G04, symbol 74xGxx:74AHCT1G04
- added U? (x2): 74AHC1G08, symbol 74xGxx:74AHC1G08
- added U?: 4081, symbol 4xxx:4081
- added U?: CLK, symbol newlib:CLK
Connections:
- net +5V: now also C?.2, R?.1, R?.2
- net GND: now also U?.6 (THR), C?.1, C?.1, C?.2, C?.2, SW?.2, U?.3 (GND), U?.3 (GND), U?.3 (GND), U?.3 (GND)
- net at U?.2 (TR), U?.6 (THR): now also R?.1, C?.2; no longer R?.2
- net at U?.3 (Q): now also U?.2
- net at U?.4 (R): now also U?.~
- net at U?.5 (CV): now also C?.1 (x2)
- net at R?.2, U?.7 (DIS): now also R?.1; no longer R?.1
- net at U?.2 (TR): now also R?.2, U?.4 (R), SW?.1
- net at U?.3 (Q): now also U?.1
- net at U?.5 (CV): now also C?.2
- net at U?.6 (THR): now also U?.7 (DIS), C?.1, R?.2
- net at U?.2 (TR): now also SW?.1 (A)
- net at U?.3 (Q): now also U?.2, U?.2
- net at U?.4 (R): now also SW?.3 (C)
- net at U?.7 (DIS): now also U?.~
- new net: R?.2, R?.2
- new net: R?.1, SW?.2 (B)
- new net: U?.1, U?.4 (x2)
- new net: U?.2, U?.4
- new net: U?.4, U?.~
- new net VCC: U?.5 (VCC), U?.5 (VCC), U?.5 (VCC), U?.5 (VCC)
Other:
- note added: "Dual AND-Gate is better to use here.\n"
- note added: "Oscillating Timer\nFor Showing the Program\n"
- note added: "Push-To-Advance\nFor debugging\n"
- note added: "Switch \n(RS-LATCH)"
